File: PCB-design/PyKey60.kicad_pcb (KiCad board)
At the start: 2 copper layers, 348.7 x 119.4 mm, 300 parts, among them J1 USB_C_Receptacle_USB2.0, J2 Conn_01x03, SW1 SW_SPST, SW2 SW_SPDT, U1 CherryMX_LTST-A683CEGBW, U10 CherryMX_LTST-A683CEGBW, U11 CherryMX_LTST-A683CEGBW, U12 CherryMX_LTST-A683CEGBW, U13 CherryMX_LTST-A683CEGBW, U14 CherryMX_LTST-A683CEGBW, U15 CherryMX_LTST-A683CEGBW, U16 CherryMX_LTST-A683CEGBW, U17 CherryMX_LTST-A683CEGBW, U18 CherryMX_LTST-A683CEGBW, U19 CherryMX_LTST-A683CEGBW, U2 CherryMX_LTST-A683CEGBW, U20 CherryMX_LTST-A683CEGBW, U21 CherryMX_LTST-A683CEGBW, U22 CherryMX_LTST-A683CEGBW, U23 CherryMX_LTST-A683CEGBW, U24 CherryMX_LTST-A683CEGBW, U25 CherryMX_LTST-A683CEGBW, U26 CherryMX_LTST-A683CEGBW, U27 CherryMX_LTST-A683CEGBW, U28 CherryMX_LTST-A683CEGBW, U29 CherryMX_LTST-A683CEGBW, U3 CherryMX_LTST-A683CEGBW, U30 CherryMX_LTST-A683CEGBW, U31 CherryMX_LTST-A683CEGBW, U32 CherryMX_LTST-A683CEGBW, U33 CherryMX_LTST-A683CEGBW, U34 CherryMX_LTST-A683CEGBW, U35 CherryMX_LTST-A683CEGBW, U36 CherryMX_LTST-A683CEGBW, U37 CherryMX_LTST-A683CEGBW, U38 CherryMX_LTST-A683CEGBW, U39 CherryMX_LTST-A683CEGBW, U4 CherryMX_LTST-A683CEGBW, U40 CherryMX_LTST-A683CEGBW, U41 CherryMX_LTST-A683CEGBW, U42 CherryMX_LTST-A683CEGBW, U43 CherryMX_LTST-A683CEGBW, U44 CherryMX_LTST-A683CEGBW, U45 CherryMX_LTST-A683CEGBW, U46 CherryMX_LTST-A683CEGBW, U47 CherryMX_LTST-A683CEGBW, U48 CherryMX_LTST-A683CEGBW, U49 CherryMX_LTST-A683CEGBW, U5 CherryMX_LTST-A683CEGBW, U50 CherryMX_LTST-A683CEGBW, U51 CherryMX_LTST-A683CEGBW, U52 CherryMX_LTST-A683CEGBW, U53 CherryMX_LTST-A683CEGBW, U54 CherryMX_LTST-A683CEGBW, U55 CherryMX_LTST-A683CEGBW, U56 CherryMX_LTST-A683CEGBW, U57 CherryMX_LTST-A683CEGBW, U58 CherryMX_LTST-A683CEGBW, U59 CherryMX_LTST-A683CEGBW, U6 CherryMX_LTST-A683CEGBW, U60 CherryMX_LTST-A683CEGBW, U61 CherryMX_LTST-A683CEGBW, U62 CherryMX_LTST-A683CEGBW, U62 RP2040, U63 CherryMX_LTST-A683CEGBW, U63 USBLC6-2SC6, U64 CherryMX_LTST-A683CEGBW, U64 W25Q128JVS, U65 AMS1117-3.3, U65 CherryMX_LTST-A683CEGBW, U66 CherryMX_LTST-A683CEGBW, U67 CherryMX_LTST-A683CEGBW, U68 CherryMX_LTST-A683CEGBW, U69 CherryMX_LTST-A683CEGBW, U7 CherryMX_LTST-A683CEGBW, U70 CherryMX_LTST-A683CEGBW, U71 CherryMX_LTST-A683CEGBW, U72 CherryMX_LTST-A683CEGBW, U73 CherryMX_LTST-A683CEGBW, U74 CherryMX_LTST-A683CEGBW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

Commit message: Move USB
Move USB and update silkscreen info (name, source URL)
Parts:
- moved R1 30.4 mm to (79.1, 41.3), turned to 0 degrees
- moved J1 26.5 mm to (88.4, 42.5)
- moved R2 26.5 mm to (97.5, 41.9), turned to 180 degrees
Routing:
- net /USB-: track 24.0 -> 53.8 mm, vias 0 -> 2
- net VBUS: track 78.5 -> 107.0 mm, vias 3 -> 5
- net /USB+: track 23.4 -> 51.9 mm, vias 0 -> 2
- net Net-(J1-PadB5): track 20.5 -> 12.0 mm
- net Net-(J1-PadA5): track 20.2 -> 12.2 mm
- net Net-(U66-Pad5): track 33.0 -> 35.7 mm, vias 0 -> 2
- net ROW2: track 655.5 -> 657.9 mm
- net +3V3: track 2543.5 -> 2544.4 mm, vias 66 -> 68
- net Net-(U1-Pad5): track 14.0 -> 13.9 mm, vias 2 -> 0
- net GND: vias 142 -> 124
Other:
- board text added: "PyKey87 TKL Keyboard RP2040 Runs Python"
- board text added: "https://github.com/nitronarcosis/PyKey87"
- board text removed: "GND 3V3 SCK TX RX CS"
- board text removed: "GND 3V3 SDA SCL"
- board text removed: "I2C1"
- board text removed: "PyKey60 60% Keyboard RP2040 Runs Python"
- board text removed: "SPI1"
- board text removed: "https://github.com/jpconstantineau/PyKey60"

Commit message: Update Schematic to Reflect PCB
Also reroute +3.3V through 100nF capacitor before LED per https://optoelectronics.liteon.com/upload/download/DS35-2019-0032/LTST-A683CEGBW.PDF
Parts:
- moved C60 0.30 mm to (179.2, 90.3), turned to 0 degrees
Routing:
- net +3V3: track 2544.4 -> 2483.3 mm

Commit message: Reinstall LED and Speaker
I decided I like knowing when caps lock  is on and want to play Star Trek sounds on my keyboard.
Parts:
- added D101: RED, LED_SMD:LED_0603_1608Metric, B.Cu at (90.0, 116.4)
- added LS1: Speaker, Buzzer:AST1109MLTRQ, B.Cu at (220.3, 151.9)
- added R8: 1k, Resistor_SMD:R_0603_1608Metric, B.Cu at (87.0, 111.3)
- U74, U77, U80, U83, U84, U87: footprint CherryMX_PCB_KailhSocket_LTST-A683CEGBW-Rotated-HS:CherryMX_1.00u_PCB_KailhSocket_LTST-A683CEGBW-Rotated-HS -> CherryMX_PCB_KailhSocket_LTST-A683CEGBW-Rotated:CherryMX_1.00u_PCB_KailhSocket_LTST-A683CEGBW-Rotated
- moved C41 1.52 mm to (74.3, 71.0), turned to 0 degrees
- renumbered C96 to C65, C94 to C65, C93 to C65, C92 to C65, C91 to C65, C90 to C65, C89 to C65, C88 to C65, C87 to C65, C86 to C65, 103 to C65, C85 to C65, C84 to C65, C83 to C65, C82 to C65, C80 to C65, C81 to C65, C79 to C65, C78 to C65, C102 to C65, C101 to C65, C100 to C65, C98 to C65, C95 to C65, C97 to C65, C99 to C65, U62 to U100, U63 to U101, U64 to U102, U65 to U103
Connections:
- net I2C1_SCL renamed Net-(U100-Pad35)
- net SPI1_CSn renamed Net-(U100-Pad37)
- net SPI1_RX renamed Net-(U100-Pad40)
- net SPI1_SCK renamed Net-(U100-Pad38)
- U100 pad 34: I2C1_SDA -> Speaker
- U100 pad 39: SPI1_TX -> LED
Routing:
- net LED: track 0.00 -> 140.7 mm, vias 0 -> 6
- net Speaker: track 0.00 -> 54.0 mm, vias 0 -> 4
- net COL17: track 336.4 -> 346.4 mm
- net Net-(D101-Pad2): track 0.00 -> 5.23 mm
- net +3V3: track 2483.3 -> 2486.3 mm
- net GND: track 297.8 -> 296.3 mm, vias 124 -> 120
- net RGBData0: track 202.6 -> 203.7 mm
- net ROW0: track 543.3 -> 542.7 mm
Other:
- board size 348.7 x 119.4 mm -> 351 x 121.5 mm
