File: PCB-design/PyKey60.kicad_pcb (KiCad board)
At the start: 2 copper layers, 353 x 120 mm, 303 parts, among them J1 USB_C_Receptacle_USB2.0, J2 Conn_01x03, SW1 SW_SPST, SW2 SW_SPDT, U1 CherryMX_LTST-A683CEGBW, U10 CherryMX_LTST-A683CEGBW, U100 RP2040, U101 USBLC6-2SC6, U102 W25Q128JVS, U103 AMS1117-3.3, U11 CherryMX_LTST-A683CEGBW, U12 CherryMX_LTST-A683CEGBW, U13 CherryMX_LTST-A683CEGBW, U14 CherryMX_LTST-A683CEGBW, U15 CherryMX_LTST-A683CEGBW, U16 CherryMX_LTST-A683CEGBW, U17 CherryMX_LTST-A683CEGBW, U18 CherryMX_LTST-A683CEGBW, U19 CherryMX_LTST-A683CEGBW, U2 CherryMX_LTST-A683CEGBW, U20 CherryMX_LTST-A683CEGBW, U21 CherryMX_LTST-A683CEGBW, U22 CherryMX_LTST-A683CEGBW, U23 CherryMX_LTST-A683CEGBW, U24 CherryMX_LTST-A683CEGBW, U25 CherryMX_LTST-A683CEGBW, U26 CherryMX_LTST-A683CEGBW, U27 CherryMX_LTST-A683CEGBW, U28 CherryMX_LTST-A683CEGBW, U29 CherryMX_LTST-A683CEGBW, U3 CherryMX_LTST-A683CEGBW, U30 CherryMX_LTST-A683CEGBW, U31 CherryMX_LTST-A683CEGBW, U32 CherryMX_LTST-A683CEGBW, U33 CherryMX_LTST-A683CEGBW, U34 CherryMX_LTST-A683CEGBW, U35 CherryMX_LTST-A683CEGBW, U36 CherryMX_LTST-A683CEGBW, U37 CherryMX_LTST-A683CEGBW, U38 CherryMX_LTST-A683CEGBW, U39 CherryMX_LTST-A683CEGBW, U4 CherryMX_LTST-A683CEGBW, U40 CherryMX_LTST-A683CEGBW, U41 CherryMX_LTST-A683CEGBW, U42 CherryMX_LTST-A683CEGBW, U43 CherryMX_LTST-A683CEGBW, U44 CherryMX_LTST-A683CEGBW, U45 CherryMX_LTST-A683CEGBW, U46 CherryMX_LTST-A683CEGBW, U47 CherryMX_LTST-A683CEGBW, U48 CherryMX_LTST-A683CEGBW, U49 CherryMX_LTST-A683CEGBW, U5 CherryMX_LTST-A683CEGBW, U50 CherryMX_LTST-A683CEGBW, U51 CherryMX_LTST-A683CEGBW, U52 CherryMX_LTST-A683CEGBW, U53 CherryMX_LTST-A683CEGBW, U54 CherryMX_LTST-A683CEGBW, U55 CherryMX_LTST-A683CEGBW, U56 CherryMX_LTST-A683CEGBW, U57 CherryMX_LTST-A683CEGBW, U58 CherryMX_LTST-A683CEGBW, U59 CherryMX_LTST-A683CEGBW, U6 CherryMX_LTST-A683CEGBW, U60 CherryMX_LTST-A683CEGBW, U61 CherryMX_LTST-A683CEGBW, U62 CherryMX_LTST-A683CEGBW, U63 CherryMX_LTST-A683CEGBW, U64 CherryMX_LTST-A683CEGBW, U65 CherryMX_LTST-A683CEGBW, U66 CherryMX_LTST-A683CEGBW, U67 CherryMX_LTST-A683CEGBW, U68 CherryMX_LTST-A683CEGBW, U69 CherryMX_LTST-A683CEGBW, U7 CherryMX_LTST-A683CEGBW, U70 CherryMX_LTST-A683CEGBW, U71 CherryMX_LTST-A683CEGBW, U72 CherryMX_LTST-A683CEGBW, U73 CherryMX_LTST-A683CEGBW, U74 CherryMX_LTST-A683CEGBW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

Commit message: Add bottom plate and I2C
Parts:
- moved R1 2.84 mm to (80.6, 44.0)
- moved R2 2.06 mm to (97.2, 44.0)
Routing:
- net ROW0: track 535.7 -> 549.2 mm
- net COL17: track 348.0 -> 338.7 mm, vias 16 -> 14
- net (no net): track 0.00 -> 5.06 mm, vias 0 -> 2
- net GND: track 296.7 -> 300.8 mm
- net RGBData1: track 375.2 -> 371.9 mm
- net RGBData5: track 351.7 -> 354.1 mm
- net /USB-: track 53.8 -> 52.2 mm
- net Net-(U56-Pad5): track 85.0 -> 86.4 mm
- net COL14: track 268.6 -> 270.0 mm
- net ROW3: track 361.8 -> 363.2 mm
- net /USB+: track 51.9 -> 50.6 mm
- net Speaker: track 51.7 -> 50.5 mm, vias 4 -> 2
- net COL15: track 298.2 -> 299.3 mm
- net ROW1: track 463.4 -> 464.5 mm
- net /RESET: track 110.6 -> 111.5 mm
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
Commit message: Add cutout for obscured switches
Also added extra holes for feet and additional standoff
Parts:
- added H7: MountingHole_2.7mm_M2.5_Pad, MountingHole:MountingHole_2.7mm_M2.5_Pad, F.Cu at (346.4, 107.5)
- moved SW2 0.10 mm to (91.5, 106.7)
Routing:
- net GND: track 300.8 -> 300.9 mm, vias 120 -> 125

Commit message: Shrink standoffs, enlarge cutout
added an additional standoff near G/H
Parts:
- added REF**: MountingHole_2.2mm_M2_Pad, MountingHole:MountingHole_2.2mm_M2_Pad, F.Cu at (190.4, 110.0)
- H1, H2, H3, H4, H5, H6, H7: value MountingHole_2.7mm_M2.5_Pad -> MountingHole_2.2mm_M2_Pad; footprint MountingHole:MountingHole_2.7mm_M2.5_Pad -> MountingHole:MountingHole_2.2mm_M2_Pad
Other:
- board size 353 x 120 mm -> 352.5 x 120 mm
