File: PCB-design/PyKey60.sch (KiCad schematic (older format))
At the start: 303 parts, among them J1 USB_C_Receptacle_USB2.0, J2 Conn_01x03, SW1 SW_SPST, SW2 SW_SPDT, U1 CherryMX_LTST-A683CEGBW, U10 CherryMX_LTST-A683CEGBW, U100 RP2040, U101 USBLC6-2SC6, U102 W25Q128JVS, U103 AMS1117-3.3, U11 CherryMX_LTST-A683CEGBW, U12 CherryMX_LTST-A683CEGBW, U13 CherryMX_LTST-A683CEGBW, U14 CherryMX_LTST-A683CEGBW, U15 CherryMX_LTST-A683CEGBW, U16 CherryMX_LTST-A683CEGBW, U17 CherryMX_LTST-A683CEGBW, U18 CherryMX_LTST-A683CEGBW, U19 CherryMX_LTST-A683CEGBW, U2 CherryMX_LTST-A683CEGBW, U20 CherryMX_LTST-A683CEGBW, U21 CherryMX_LTST-A683CEGBW, U22 CherryMX_LTST-A683CEGBW, U23 CherryMX_LTST-A683CEGBW, U24 CherryMX_LTST-A683CEGBW, U25 CherryMX_LTST-A683CEGBW, U26 CherryMX_LTST-A683CEGBW, U27 CherryMX_LTST-A683CEGBW, U28 CherryMX_LTST-A683CEGBW, U29 CherryMX_LTST-A683CEGBW, U3 CherryMX_LTST-A683CEGBW, U30 CherryMX_LTST-A683CEGBW, U31 CherryMX_LTST-A683CEGBW, U32 CherryMX_LTST-A683CEGBW, U33 CherryMX_LTST-A683CEGBW, U34 CherryMX_LTST-A683CEGBW, U35 CherryMX_LTST-A683CEGBW, U36 CherryMX_LTST-A683CEGBW, U37 CherryMX_LTST-A683CEGBW, U38 CherryMX_LTST-A683CEGBW, U39 CherryMX_LTST-A683CEGBW, U4 CherryMX_LTST-A683CEGBW, U40 CherryMX_LTST-A683CEGBW, U41 CherryMX_LTST-A683CEGBW, U42 CherryMX_LTST-A683CEGBW, U43 CherryMX_LTST-A683CEGBW, U44 CherryMX_LTST-A683CEGBW, U45 CherryMX_LTST-A683CEGBW, U46 CherryMX_LTST-A683CEGBW, U47 CherryMX_LTST-A683CEGBW, U48 CherryMX_LTST-A683CEGBW, U49 CherryMX_LTST-A683CEGBW, U5 CherryMX_LTST-A683CEGBW, U50 CherryMX_LTST-A683CEGBW, U51 CherryMX_LTST-A683CEGBW, U52 CherryMX_LTST-A683CEGBW, U53 CherryMX_LTST-A683CEGBW, U54 CherryMX_LTST-A683CEGBW, U55 CherryMX_LTST-A683CEGBW, U56 CherryMX_LTST-A683CEGBW, U57 CherryMX_LTST-A683CEGBW, U58 CherryMX_LTST-A683CEGBW, U59 CherryMX_LTST-A683CEGBW, U6 CherryMX_LTST-A683CEGBW, U60 CherryMX_LTST-A683CEGBW, U61 CherryMX_LTST-A683CEGBW, U62 CherryMX_LTST-A683CEGBW, U63 CherryMX_LTST-A683CEGBW, U64 CherryMX_LTST-A683CEGBW, U65 CherryMX_LTST-A683CEGBW, U66 CherryMX_LTST-A683CEGBW, U67 CherryMX_LTST-A683CEGBW, U68 CherryMX_LTST-A683CEGBW, U69 CherryMX_LTST-A683CEGBW, U7 CherryMX_LTST-A683CEGBW, U70 CherryMX_LTST-A683CEGBW, U71 CherryMX_LTST-A683CEGBW, U72 CherryMX_LTST-A683CEGBW, U73 CherryMX_LTST-A683CEGBW, U74 CherryMX_LTST-A683CEGBW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

Commit message: Shrink standoffs, enlarge cutout
added an additional standoff near G/H
Parts:
- H1, H2, H3, H4, H5, H6, H7: footprint MountingHole:MountingHole_2.7mm_M2.5_Pad -> MountingHole:MountingHole_2.2mm_M2_Pad
Changed lines of the file:
@@
 F 0 "H1" H 19050 6849 50  0000 L CNN
 F 1 "MountingHole_Pad" H 19050 6758 50  0000 L CNN
-F 2 "MountingHole:MountingHole_2.7mm_M2.5_Pad" H 18950 6800 50  0001 C CNN
+F 2 "MountingHole:MountingHole_2.2mm_M2_Pad" H 18950 6800 50  0001 C CNN
 F 3 "~" H 18950 6800 50  0001 C CNN
 	1    18950 6800
@@
 F 0 "H2" H 19050 7299 50  0000 L CNN
 F 1 "MountingHole_Pad" H 19050 7208 50  0000 L CNN
-F 2 "MountingHole:MountingHole_2.7mm_M2.5_Pad" H 18950 7250 50  0001 C CNN
+F 2 "MountingHole:MountingHole_2.2mm_M2_Pad" H 18950 7250 50  0001 C CNN
 F 3 "~" H 18950 7250 50  0001 C CNN
 	1    18950 7250
@@
 F 0 "H3" H 20000 6849 50  0000 L CNN
 F 1 "MountingHole_Pad" H 20000 6758 50  0000 L CNN
-F 2 "MountingHole:MountingHole_2.7mm_M2.5_Pad" H 19900 6800 50  0001 C CNN
+F 2 "MountingHole:MountingHole_2.2mm_M2_Pad" H 19900 6800 50  0001 C CNN
 F 3 "~" H 19900 6800 50  0001 C CNN
 	1    19900 6800
@@
 F 0 "H4" H 20000 7299 50  0000 L CNN
 F 1 "MountingHole_Pad" H 20000 7208 50  0000 L CNN
-F 2 "MountingHole:MountingHole_2.7mm_M2.5_Pad" H 19900 7250 50  0001 C CNN
+F 2 "MountingHole:MountingHole_2.2mm_M2_Pad" H 19900 7250 50  0001 C CNN
 F 3 "~" H 19900 7250 50  0001 C CNN
 	1    19900 7250
@@
 F 0 "H6" H 20950 7299 50  0000 L CNN
 F 1 "MountingHole_Pad" H 20950 7208 50  0000 L CNN
-F 2 "MountingHole:MountingHole_2.7mm_M2.5_Pad" H 20850 7250 50  0001 C CNN
+F 2 "MountingHole:MountingHole_2.2mm_M2_Pad" H 20850 7250 50  0001 C CNN
 F 3 "~" H 20850 7250 50  0001 C CNN
 	1    20850 7250
@@
 F 0 "H5" H 20950 6849 50  0000 L CNN
 F 1 "MountingHole_Pad" H 20950 6758 50  0000 L CNN
-F 2 "MountingHole:MountingHole_2.7mm_M2.5_Pad" H 20850 6800 50  0001 C CNN
+F 2 "MountingHole:MountingHole_2.2mm_M2_Pad" H 20850 6800 50  0001 C CNN
 F 3 "~" H 20850 6800 50  0001 C CNN
 	1    20850 6800
@@
 F 0 "H7" H 20650 7049 50  0000 L CNN
 F 1 "MountingHole_Pad" H 20650 6958 50  0000 L CNN
-F 2 "MountingHole:MountingHole_2.7mm_M2.5_Pad" H 20550 7000 50  0001 C CNN
+F 2 "MountingHole:MountingHole_2.2mm_M2_Pad" H 20550 7000 50  0001 C CNN
 F 3 "~" H 20550 7000 50  0001 C CNN
 	1    20550 7000
