File: Bottom-plate/PyKey87-bottom/PyKey87-bottom.kicad_pcb (KiCad board)
At the start: 2 copper layers, 353 x 120 mm, 8 parts

Commit message: Add cutout for obscured switches
Also added extra holes for feet and additional standoff
Parts:
- added H7: MountingHole_Pad, MountingHole:MountingHole_2.7mm_Pad, F.Cu at (346.4, 107.5)
- renumbered H7 to H8, H8 to H9
Other:
- outline, holes or cut-outs redrawn
- board text added: "Reset"
- board text added: "Run Boot"
Changed lines of the file:
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@@
   (general
     (thickness 1.6)
-    (drawings 8)
+    (drawings 14)
     (tracks 0)
     (zones 0)
-    (modules 8)
-    (nets 9)
+    (modules 9)
+    (nets 10)
   )
   (page A4)
@@
     (solder_mask_min_width 0.25)
     (aux_axis_origin 0 0)
-    (visible_elements FFFFFF7F)
+    (visible_elements 7FFFFFFF)
     (pcbplotparams
       (layerselection 0x010fc_ffffffff)
@@
   (net 7 "Net-(H7-Pad1)")
   (net 8 "Net-(H8-Pad1)")
+  (net 9 "Net-(H9-Pad1)")
   (net_class Default "This is the default net class."
     (clearance 0.2)
@@
     (add_net "Net-(H7-Pad1)")
     (add_net "Net-(H8-Pad1)")
+    (add_net "Net-(H9-Pad1)")
+  )
+  (module MountingHole:MountingHole_2.7mm_Pad (layer F.Cu)
+    (at 346.375 107.475)
+    (descr "Mounting Hole 2.7mm")
+    (tags "mounting hole 2.7mm")
+    (attr virtual)
+    (fp_text reference H7 (at 0 -3.7) (layer F.SilkS)
+      (effects (font (size 1 1) (thickness 0.15)))
+    )
+    (fp_text value MountingHole_Pad (at 0 3.7) (layer F.Fab)
+      (effects (font (size 1 1) (thickness 0.15)))
+    )
+    (fp_circle (center 0 0) (end 2.95 0) (layer F.CrtYd) (width 0.05))
+    (fp_circle (center 0 0) (end 2.7 0) (layer Cmts.User) (width 0.15))
+    (fp_text user %R (at 0.3 0) (layer F.Fab)
+      (effects (font (size 1 1) (thickness 0.15)))
+    )
+    (pad 1 thru_hole circle (at 0 0) (size 5.4 5.4) (drill 2.7) (layers *.Cu *.Mask)
+      (net 9 "Net-(H9-Pad1)"))
   )
   (module MountingHole:MountingHole_4.3mm_M4_Pad (layer F.Cu)
@@
     (tags "mounting hole 4.3mm m4")
     (attr virtual)
-    (fp_text reference H8 (at 0 -5.3) (layer F.SilkS)
+    (fp_text reference H9 (at 0 -5.3) (layer F.SilkS)
       (effects (font (size 1 1) (thickness 0.15)))
     )
@@
     (tags "mounting hole 4.3mm m4")
     (attr virtual)
-    (fp_text reference H7 (at 0 -5.3) (layer F.SilkS)
+    (fp_text reference H8 (at 0 -5.3) (layer F.SilkS)
       (effects (font (size 1 1) (thickness 0.15)))
     )
@@
       (net 1 "Net-(H1-Pad1)"))
   )
+  (gr_text Reset (at 91.44 115.57) (layer B.Cu)
+    (effects (font (size 1 1) (thickness 0.15)) (justify mirror))
+  )
+  (gr_text "Run    Boot" (at 91.44 104.14) (layer B.Cu)
+    (effects (font (size 1 1) (thickness 0.15)) (justify mirror))
+  )
+  (gr_line (start 95 106) (end 88 106) (layer Edge.Cuts) (width 0.12))
+  (gr_line (start 95 114) (end 95 106) (layer Edge.Cuts) (width 0.12))
+  (gr_line (start 88 114) (end 95 114) (layer Edge.Cuts) (width 0.12))
+  (gr_line (start 88 106) (end 88 114) (layer Edge.Cuts) (width 0.12))
   (gr_arc (start 61 158) (end 61 160) (angle 90) (layer Edge.Cuts) (width 0.09906))
   (gr_arc (start 60.96 42) (end 58.96 42) (angle 90) (layer Edge.Cuts) (width 0.09906))

Commit message: Shrink standoffs, enlarge cutout
added an additional standoff near G/H
Parts:
- added REF**: LED_0603_1608Metric, LED_SMD:LED_0603_1608Metric, F.Cu at (90.0, 116.4)
- added REF**: SW_Push_SPST_NO_Alps_SKRK, Button_Switch_SMD:SW_Push_SPST_NO_Alps_SKRK, F.Cu at (91.5, 112.6)
- added REF**: SW_SPDT_PCM12, Button_Switch_SMD:SW_SPDT_PCM12, F.Cu at (91.5, 106.7)
- H1, H2, H3, H4, H5, H6, H7: footprint MountingHole:MountingHole_2.7mm_Pad -> MountingHole:MountingHole_2.2mm_M2_Pad
Other:
- outline, holes or cut-outs redrawn
