File: pykey87/PCB-design/PyKey87.kicad_pcb (KiCad board)
At the start: 2 copper layers, 352.5 x 120 mm, 305 parts, among them J1 USB_C_Receptacle_USB2.0, J2 Conn_01x03, SW1 SW_SPST, SW2 SW_SPDT, U1 CherryMX_LTST-A683CEGBW, U10 CherryMX_LTST-A683CEGBW, U100 RP2040, U101 USBLC6-2SC6, U102 W25Q128JVS, U103 AMS1117-3.3, U11 CherryMX_LTST-A683CEGBW, U12 CherryMX_LTST-A683CEGBW, U13 CherryMX_LTST-A683CEGBW, U14 CherryMX_LTST-A683CEGBW, U15 CherryMX_LTST-A683CEGBW, U16 CherryMX_LTST-A683CEGBW, U17 CherryMX_LTST-A683CEGBW, U18 CherryMX_LTST-A683CEGBW, U19 CherryMX_LTST-A683CEGBW, U2 CherryMX_LTST-A683CEGBW, U20 CherryMX_LTST-A683CEGBW, U21 CherryMX_LTST-A683CEGBW, U22 CherryMX_LTST-A683CEGBW, U23 CherryMX_LTST-A683CEGBW, U24 CherryMX_LTST-A683CEGBW, U25 CherryMX_LTST-A683CEGBW, U26 CherryMX_LTST-A683CEGBW, U27 CherryMX_LTST-A683CEGBW, U28 CherryMX_LTST-A683CEGBW, U29 CherryMX_LTST-A683CEGBW, U3 CherryMX_LTST-A683CEGBW, U30 CherryMX_LTST-A683CEGBW, U31 CherryMX_LTST-A683CEGBW, U32 CherryMX_LTST-A683CEGBW, U33 CherryMX_LTST-A683CEGBW, U34 CherryMX_LTST-A683CEGBW, U35 CherryMX_LTST-A683CEGBW, U36 CherryMX_LTST-A683CEGBW, U37 CherryMX_LTST-A683CEGBW, U38 CherryMX_LTST-A683CEGBW, U39 CherryMX_LTST-A683CEGBW, U4 CherryMX_LTST-A683CEGBW, U40 CherryMX_LTST-A683CEGBW, U41 CherryMX_LTST-A683CEGBW, U42 CherryMX_LTST-A683CEGBW, U43 CherryMX_LTST-A683CEGBW, U44 CherryMX_LTST-A683CEGBW, U45 CherryMX_LTST-A683CEGBW, U46 CherryMX_LTST-A683CEGBW, U47 CherryMX_LTST-A683CEGBW, U48 CherryMX_LTST-A683CEGBW, U49 CherryMX_LTST-A683CEGBW, U5 CherryMX_LTST-A683CEGBW, U50 CherryMX_LTST-A683CEGBW, U51 CherryMX_LTST-A683CEGBW, U52 CherryMX_LTST-A683CEGBW, U53 CherryMX_LTST-A683CEGBW, U54 CherryMX_LTST-A683CEGBW, U55 CherryMX_LTST-A683CEGBW, U56 CherryMX_LTST-A683CEGBW, U57 CherryMX_LTST-A683CEGBW, U58 CherryMX_LTST-A683CEGBW, U59 CherryMX_LTST-A683CEGBW, U6 CherryMX_LTST-A683CEGBW, U60 CherryMX_LTST-A683CEGBW, U61 CherryMX_LTST-A683CEGBW, U62 CherryMX_LTST-A683CEGBW, U63 CherryMX_LTST-A683CEGBW, U64 CherryMX_LTST-A683CEGBW, U65 CherryMX_LTST-A683CEGBW, U66 CherryMX_LTST-A683CEGBW, U67 CherryMX_LTST-A683CEGBW, U68 CherryMX_LTST-A683CEGBW, U69 CherryMX_LTST-A683CEGBW, U7 CherryMX_LTST-A683CEGBW, U70 CherryMX_LTST-A683CEGBW, U71 CherryMX_LTST-A683CEGBW, U72 CherryMX_LTST-A683CEGBW, U73 CherryMX_LTST-A683CEGBW, U74 CherryMX_LTST-A683CEGBW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

Commit message: Moving things around
Prep for merging. Also did some clean up and added 8th standoff.
Parts:
- added REF**: MountingHole_1.152mm, lib.pretty:MountingHole_1.152mm, F.Cu at (61.9, 42.4)
- renumbered REF** to H8
Routing:
- net GND: vias 125 -> 129
Other:
- board text added: "CERN-OHL-W 2021-11-?? - Pierre Constantineau & nitronarcosis"
- board text added: "https://github.com/jpconstantineau/PyKey60"
- board text removed: "CERN-OHL-W 2021-09-01 - Pierre Constantineau"
- board text removed: "https://github.com/nitronarcosis/PyKey87"
Changed lines of the file:
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@@
     (thickness 1.6002)
     (drawings 93)
-    (tracks 3663)
+    (tracks 3669)
     (zones 0)
-    (modules 305)
+    (modules 306)
     (nets 231)
   )
@@
     (0 Front signal)
     (31 Back signal)
-    (32 B.Adhes user)
+    (32 B.Adhes user hide)
     (33 F.Adhes user)
     (34 B.Paste user)
@@
     (37 F.SilkS user)
     (38 B.Mask user)
-    (39 F.Mask user)
+    (39 F.Mask user hide)
     (40 Dwgs.User user hide)
-    (41 Cmts.User user)
+    (41 Cmts.User user hide)
     (42 Eco1.User user hide)
-    (43 Eco2.User user)
+    (43 Eco2.User user hide)
     (44 Edge.Cuts user)
     (45 Margin user)
@@
     (mod_text_size 1.524 1.524)
     (mod_text_width 0.3048)
-    (pad_size 0.875 0.2)
-    (pad_drill 0)
+    (pad_size 1.152 1.152)
+    (pad_drill 1.152)
     (pad_to_mask_clearance 0.0762)
     (aux_axis_origin 66.675 83.345)
@@
     (uvia_drill 0.127)
   )
+  (module lib.pretty:MountingHole_1.152mm (layer Front)
+    (at 61.895 42.405)
+    (descr "Mounting Hole 2.1mm, no annular")
+    (tags "mounting hole 2.1mm no annular")
+    (attr virtual)
+    (fp_text reference REF** (at 0 -3.2) (layer F.SilkS)
+      (effects (font (size 1 1) (thickness 0.15)))
+    )
+    (fp_text value MountingHole_1.152mm (at 0 3.2) (layer F.Fab)
+      (effects (font (size 1 1) (thickness 0.15)))
+    )
+    (fp_circle (center 0 0) (end 2.35 0) (layer F.CrtYd) (width 0.05))
+    (fp_circle (center 0 0) (end 2.1 0) (layer Cmts.User) (width 0.15))
+    (fp_text user %R (at 0.3 0) (layer F.Fab)
+      (effects (font (size 1 1) (thickness 0.15)))
+    )
+    (pad "" np_thru_hole circle (at 0 0) (size 1.152 1.152) (drill 1.152) (layers *.Cu *.Mask)
+      (solder_mask_margin 0.148) (solder_paste_margin 1.152) (zone_connect 0))
+  )
   (module MountingHole:MountingHole_2.2mm_M2_Pad (layer Front)
     (at 190.365 110.015)
@@
     (tags "mounting hole 2.2mm m2")
     (attr virtual)
-    (fp_text reference REF** (at 0 -3.2) (layer F.SilkS)
+    (fp_text reference H8 (at 0 -3.2) (layer F.SilkS)
       (effects (font (size 1 1) (thickness 0.15)))
     )
@@
   (gr_arc (start 61.5 42) (end 61.5 40) (angle -90) (layer Edge.Cuts) (width 0.1))
   (gr_line (start 61.5 40) (end 410 40) (angle 90) (layer Edge.Cuts) (width 0.09906))
-  (gr_text https://github.com/nitronarcosis/PyKey87 (at 222.885 143.035) (layer B.SilkS)
+  (gr_text https://github.com/jpconstantineau/PyKey60 (at 222.885 143.035) (layer B.SilkS)
     (effects (font (size 1 1) (thickness 0.15)) (justify mirror))
   )
@@
     (effects (font (size 1 1) (thickness 0.1)) (justify mirror))
   )
-  (gr_text "CERN-OHL-W\n2021-09-01 - Pierre Constantineau" (at 307.594 140.495) (layer B.SilkS)
+  (gr_text "CERN-OHL-W\n2021-11-?? - Pierre Constantineau & nitronarcosis" (at 307.594 140.495) (layer B.SilkS)
     (effects (font (size 1.524 1.524) (thickness 0.3048)) (justify left mirror))
   )
@@
   (segment (start 90.69 105.283) (end 90.805 105.398) (width 0.1524) (layer Back) (net 61))
   (segment (start 90.805 105.398) (end 90.805 110.777) (width 0.1524) (layer Back) (net 61))
+  (via (at 302.895 125.255) (size 0.6096) (drill 0.3048) (layers Front Back) (net 61))
+  (via (at 306.705 45.245) (size 0.6096) (drill 0.3048) (layers Front Back) (net 61))
+  (via (at 346.075 45.245) (size 0.6096) (drill 0.3048) (layers Front Back) (net 61))
+  (via (at 387.985 45.245) (size 0.6096) (drill 0.3048) (layers Front Back) (net 61))
   (segment (start 97.928 125.763) (end 95.275 128.416) (width 0.889) (layer Back) (net 62) (status 20))
   (segment (start 98.399 125.763) (end 97.928 125.763) (width 0.889) (layer Back) (net 62) (status 10))
@@
   (segment (start 197.075 107.82) (end 194.80741 107.82) (width 0.1524) (layer Back) (net 136) (status 10))
   (via (at 194.71641 107.729) (size 0.6096) (drill 0.3048) (layers Front Back) (net 136))
-  (segment (start 186.69 106.078) (end 188.341 107.729) (width 0.1524) (layer Front) (net 136))
-  (segment (start 188.341 107.729) (end 194.71641 107.729) (width 0.1524) (layer Front) (net 136))
+  (segment (start 193.929 107.729) (end 194.71641 107.729) (width 0.1524) (layer Front) (net 136))
+  (segment (start 192.405 106.205) (end 193.929 107.729) (width 0.1524) (layer Front) (net 136))
+  (segment (start 186.69 106.078) (end 186.817 106.205) (width 0.1524) (layer Front) (net 136))
+  (segment (start 186.817 106.205) (end 192.405 106.205) (width 0.1524) (layer Front) (net 136))
   (via (at 205.613 105.824) (size 0.6096) (drill 0.3048) (layers Front Back) (net 137))
   (segment (start 205.517 105.92) (end 205.613 105.824) (width 0.1524) (layer Back) (net 137))

Commit message: Added I2C header
and 2nd tooling hole
Parts:
- added REF**: JST_SH_SM04B-SRSS-TB_1x04-1MP_P1.00mm_Horizontal, Connector_JST:JST_SH_SM04B-SRSS-TB_1x04-1MP_P1.00mm_Horizontal, B.Cu at (249.6, 151.9)
- added REF**: MountingHole_1.152mm, lib.pretty:MountingHole_1.152mm, F.Cu at (409.6, 157.5)
Routing:
- net (no net): track 5.06 -> 172.9 mm, vias 2 -> 4
- net +3V3: track 2487.0 -> 2518.6 mm, vias 68 -> 69
- net GND: track 300.9 -> 304.3 mm, vias 129 -> 130
- net Speaker: track 50.5 -> 49.7 mm

Commit message: Move boot/run and reset to edge
Also cleanup, renaming, and adding a second I2C header.
Parts:
- added ?: PinHeader_1x04_P2.54mm_Vertical, Connector_PinHeader_2.54mm:PinHeader_1x04_P2.54mm_Vertical, F.Cu at (360.0, 115.1)
- H7: value MountingHole -> MountingHole_Pad
- moved SW1 75.0 mm to (118.7, 42.7), turned to 270 degrees
- moved SW2 63.6 mm to (97.9, 43.5), turned to 0 degrees
- moved R2 5.20 mm to (92.6, 46.5), turned to 90 degrees
- moved J1 2.00 mm to (86.4, 44.0)
- moved R1 1.80 mm to (79.4, 42.7), turned to 90 degrees
- renumbered H5 to ?, H1 to ?, H4 to ?, REF** to ?, H8 to ?, H7 to ?, H3 to ?, H6 to ?, H2 to ?, C41 to C42, REF** to J3
Connections:
- J3 pad 3: (no net) -> I2C1_SDA
- J3 pad 4: (no net) -> I2C1_SCL
- U100 pad 34: (no net) -> I2C1_SDA
- U100 pad 35: (no net) -> I2C1_SCL
- U100 pad 38: (no net) -> Net-(U100-Pad38)
- U100 pad 40: (no net) -> Net-(U100-Pad40)
Routing:
- net I2C1_SCL: track 0.00 -> 234.2 mm, vias 0 -> 4
- net I2C1_SDA: track 0.00 -> 233.8 mm, vias 0 -> 4
- net (no net): track 172.9 -> 0.00 mm, vias 4 -> 0
- net /RESET: track 111.5 -> 156.9 mm, vias 2 -> 6
- net Net-(R7-Pad2): track 100.6 -> 136.6 mm, vias 2 -> 4
- net GND: track 304.3 -> 316.7 mm, vias 130 -> 140
- net +3V3: track 2518.6 -> 2528.6 mm, vias 69 -> 71
- net COL3: track 183.5 -> 188.7 mm
- net COL6: track 160.2 -> 163.4 mm
- net COL4: track 138.1 -> 140.9 mm
- net COL14: track 270.0 -> 268.0 mm
- net /USB+: track 50.6 -> 48.9 mm
- net Net-(U63-Pad5): track 13.9 -> 15.4 mm
- net COL13: track 240.4 -> 239.1 mm
- net Net-(J1-PadA5): track 13.5 -> 12.2 mm
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