File: pykey87/PCB-design/PyKey87.kicad_pcb (KiCad board)
At the start: 2 copper layers, 352.5 x 120 mm, 310 parts, among them J1 USB_C_Receptacle_USB2.0, J2 Conn_01x03, J3 Conn_01x04, J4 AudioJack4, J5 Conn_01x04, SW1 SW_SPST, SW2 SW_SPDT, U1 CherryMX_LTST-A683CEGBW, U10 CherryMX_LTST-A683CEGBW, U100 RP2040, U101 USBLC6-2SC6, U102 W25Q128JVS, U103 AMS1117-3.3, U11 CherryMX_LTST-A683CEGBW, U12 CherryMX_LTST-A683CEGBW, U13 CherryMX_LTST-A683CEGBW, U14 CherryMX_LTST-A683CEGBW, U15 CherryMX_LTST-A683CEGBW, U16 CherryMX_LTST-A683CEGBW, U17 CherryMX_LTST-A683CEGBW, U18 CherryMX_LTST-A683CEGBW, U19 CherryMX_LTST-A683CEGBW, U2 CherryMX_LTST-A683CEGBW, U20 CherryMX_LTST-A683CEGBW, U21 CherryMX_LTST-A683CEGBW, U22 CherryMX_LTST-A683CEGBW, U23 CherryMX_LTST-A683CEGBW, U24 CherryMX_LTST-A683CEGBW, U25 CherryMX_LTST-A683CEGBW, U26 CherryMX_LTST-A683CEGBW, U27 CherryMX_LTST-A683CEGBW, U28 CherryMX_LTST-A683CEGBW, U29 CherryMX_LTST-A683CEGBW, U3 CherryMX_LTST-A683CEGBW, U30 CherryMX_LTST-A683CEGBW, U31 CherryMX_LTST-A683CEGBW, U32 CherryMX_LTST-A683CEGBW, U33 CherryMX_LTST-A683CEGBW, U34 CherryMX_LTST-A683CEGBW, U35 CherryMX_LTST-A683CEGBW, U36 CherryMX_LTST-A683CEGBW, U37 CherryMX_LTST-A683CEGBW, U38 CherryMX_LTST-A683CEGBW, U39 CherryMX_LTST-A683CEGBW, U4 CherryMX_LTST-A683CEGBW, U40 CherryMX_LTST-A683CEGBW, U41 CherryMX_LTST-A683CEGBW, U42 CherryMX_LTST-A683CEGBW, U43 CherryMX_LTST-A683CEGBW, U44 CherryMX_LTST-A683CEGBW, U45 CherryMX_LTST-A683CEGBW, U46 CherryMX_LTST-A683CEGBW, U47 CherryMX_LTST-A683CEGBW, U48 CherryMX_LTST-A683CEGBW, U49 CherryMX_LTST-A683CEGBW, U5 CherryMX_LTST-A683CEGBW, U50 CherryMX_LTST-A683CEGBW, U51 CherryMX_LTST-A683CEGBW, U52 CherryMX_LTST-A683CEGBW, U53 CherryMX_LTST-A683CEGBW, U54 CherryMX_LTST-A683CEGBW, U55 CherryMX_LTST-A683CEGBW, U56 CherryMX_LTST-A683CEGBW, U57 CherryMX_LTST-A683CEGBW, U58 CherryMX_LTST-A683CEGBW, U59 CherryMX_LTST-A683CEGBW, U6 CherryMX_LTST-A683CEGBW, U60 CherryMX_LTST-A683CEGBW, U61 CherryMX_LTST-A683CEGBW, U62 CherryMX_LTST-A683CEGBW, U63 CherryMX_LTST-A683CEGBW, U64 CherryMX_LTST-A683CEGBW, U65 CherryMX_LTST-A683CEGBW, U66 CherryMX_LTST-A683CEGBW, U67 CherryMX_LTST-A683CEGBW, U68 CherryMX_LTST-A683CEGBW, U69 CherryMX_LTST-A683CEGBW, U7 CherryMX_LTST-A683CEGBW, U70 CherryMX_LTST-A683CEGBW, U71 CherryMX_LTST-A683CEGBW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

Commit message: Initial upload of plate, fixing issues
Parts:
- moved D87 14.8 mm to (391.1, 149.4), turned to 90 degrees
- moved D84 4.02 mm to (391.8, 135.4), turned to 90 degrees
- moved D85 3.39 mm to (372.1, 154.5), turned to 90 degrees
- moved D86 3.39 mm to (391.1, 154.5), turned to 90 degrees
- moved U101 3.37 mm to (88.3, 86.1)
- turned SW1 to 180 degrees
Connections:
- D87 pad 1: ROW5 -> Net-(D86-Pad2)
Routing:
- net Net-(D87-Pad2): track 4.07 -> 23.2 mm
- net ROW5: track 334.9 -> 321.6 mm
- net GND: track 297.6 -> 289.2 mm, vias 140 -> 143
- net VBUS: track 111.6 -> 103.3 mm, vias 3 -> 2
- net ROW4: track 364.0 -> 369.3 mm
- net +3V3: track 2535.1 -> 2537.0 mm
- net I2C1_SDA: track 345.4 -> 346.9 mm
- net /USB+: track 49.7 -> 48.3 mm
- net Data-: track 114.7 -> 116.1 mm
- net Data+: track 113.5 -> 114.9 mm
- net Net-(D85-Pad2): track 4.04 -> 2.82 mm
- net /USB-: track 49.1 -> 48.2 mm
- net /RESET: track 146.8 -> 146.0 mm
- net Net-(D86-Pad2): track 4.04 -> 4.60 mm
- net Net-(D84-Pad2): track 4.04 -> 3.49 mm

Commit message: Update PyKey87.kicad_pcb
Routing:
- net /USB-: track 48.2 -> 44.1 mm
- net ROW0: track 565.6 -> 567.5 mm
- net /USB+: track 48.3 -> 49.9 mm
- net GND: vias 143 -> 145

Commit message: Move D87 for better fit
Parts:
- moved D86 6.62 mm to (389.3, 148.1)
- moved D87 1.44 mm to (391.8, 148.1)
Connections:
- D87 pad 1: Net-(D86-Pad2) -> ROW5
Routing:
- net ROW5: track 321.6 -> 331.1 mm
- net Net-(D86-Pad2): track 4.60 -> 6.88 mm
- net +3V3: track 2536.8 -> 2535.8 mm
- net Net-(U86-Pad5): track 13.9 -> 14.8 mm
- net I2C1_SDA: track 346.9 -> 347.6 mm
- net GND: vias 145 -> 146
