File: pykey87/Switch-plate/Switch-plate.kicad_pcb (KiCad board)
At the start: 2 copper layers, 352.7 x 120.1 mm, 0 parts

Commit message: Move D87 for better fit
Other:
- board size 352.7 x 120.1 mm -> 352.5 x 120 mm

Commit message: Misc fixes to schematic, PCB, and plates
Routing:
- added copper zone on B.Cu, net (none)
- added copper zone on F.Cu, net (none)
Other:
- outline, holes or cut-outs redrawn

Commit message: Moved Row0, and rotated stabilizers in plate
Other:
- outline, holes or cut-outs redrawn

Commit message: Refill switch plate and generate gerbers
Routing:
- added copper zone on B.Cu, net GND
- added copper zone on F.Cu, net GND
- removed copper zone on B.Cu, net (none)
- removed copper zone on F.Cu, net (none)
Changed lines of the file:
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@@
     (zones 0)
     (modules 0)
-    (nets 1)
+    (nets 2)
   )
   (page A4)
@@
   )
   (net 0 "")
+  (net 1 GND)
   (net_class Default "This is the default net class."
     (clearance 0.2)
@@
   (gr_line (start 64.975 56.525) (end 77.975 56.525) (layer Edge.Cuts) (width 0.1))
   (gr_line (start 64.975 42.525) (end 77.975 42.525) (layer Edge.Cuts) (width 0.1))
-  (zone (net 0) (net_name "") (layer B.Cu) (hatch edge 0.508)
+  (zone (net 1) (net_name GND) (layer F.Cu) (hatch edge 0.508)
     (connect_pads (clearance 0.508))
     (min_thickness 0.254)
@@
     (polygon
       (pts
-        (xy 416.56 162.56) (xy 57.15 162.56) (xy 57.15 38.1) (xy 415.29 38.1)
+        (xy 414.02 162.56) (xy 57.15 162.56) (xy 57.15 36.83) (xy 414.02 36.83)
       )
     )
   )
-  (zone (net 0) (net_name "") (layer F.Cu) (hatch edge 0.508)
+  (zone (net 1) (net_name GND) (layer B.Cu) (hatch edge 0.508)
     (connect_pads (clearance 0.508))
     (min_thickness 0.254)
@@
     (polygon
       (pts
-        (xy 416.56 162.56) (xy 57.15 162.56) (xy 57.15 38.1) (xy 415.29 38.1)
+        (xy 414.02 162.56) (xy 57.15 162.56) (xy 57.15 36.83) (xy 414.02 36.83)
       )
     )
