File: pykey18/switch-plate/PyKey18/PyKey18.kicad_pcb (KiCad board)
At the start: 2 copper layers, 81 x 120 mm, 84 parts, among them J1 USB_C_Receptacle_USB2.0, J2 Conn_01x03, J3 Conn_01x04, J4 AudioJack4, J5 Conn_01x04, SW101 SW_SPST, SW2 SW_SPDT, SW4 Rotary_Encoder_Switch, U1 CherryMX_LTST-A683CEGBW, U10 CherryMX_LTST-A683CEGBW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

Commit message: updates to pykey87
Parts:
- removed C101, C102, C103, C104, C105, C106, C107, C108, C109, C110: 100n, Capacitor_SMD:C_0603_1608Metric
- removed C111, C112: 1u, Capacitor_SMD:C_0603_1608Metric
- removed C113, C116: 22p, Capacitor_SMD:C_0603_1608Metric
- removed C114, C115: 22u, Capacitor_SMD:C_0603_1608Metric
- removed D1, D10, D11, D12, D13, D14, D15, D16, D17, D18, D2, D3, D4, D5, D6, D7, D8, D9: D, Diode_SMD:D_SOD-123
- removed D101: RED, LED_SMD:LED_0603_1608Metric
- removed H1, H2, H3, H4: MountingHole, MountingHole:MountingHole_2.2mm_M2_DIN965
- removed H10, H11: PCBA, JLCPCBA:PCBA Hole
- removed H5, H6: MountingHole-feet, MountingHole:MountingHole_4.3mm_M4
- removed H7: Logo, lib:KB_BlueMicro
- removed H8, H9: Stabs, CherryMX_StabWireBottom:CherryMX_2.00u_StabWireBottom-nokey
- removed J1: USB_C_Receptacle_USB2.0, Connector_USB:USB_C_Receptacle_HRO_TYPE-C-31-M-12
- removed J2: Conn_01x03, Connector_PinHeader_2.54mm:PinHeader_1x03_P2.54mm_Vertical
- removed J3: Conn_01x04, Connector_JST:JST_SH_SM04B-SRSS-TB_1x04-1MP_P1.00mm_Horizontal
- removed J4: AudioJack4, Connector_Audio:Jack_3.5mm_PJ320D_Horizontal
- removed J5: Conn_01x04, Connector_PinHeader_2.54mm:PinHeader_1x04_P2.54mm_Vertical
- removed LS1: Speaker, Buzzer_Beeper:Buzzer_Mallory_AST1109MLTRQ
- removed R1, R2: 5.1k, Resistor_SMD:R_0603_1608Metric
- removed R3: DNP, Resistor_SMD:R_0603_1608Metric
- removed R4, R7, R8: 1k, Resistor_SMD:R_0603_1608Metric
- removed R5, R6: 22, Resistor_SMD:R_0603_1608Metric
- removed SW101: SW_SPST, Button_Switch_SMD:Panasonic_EVQPUL_EVQPUC
- removed SW2: SW_SPDT, Button_Switch_SMD:SW_SPDT_PCM12
- removed SW4: Rotary_Encoder_Switch, Rotary_Encoder:RotaryEncoder_Alps_EC11E-Switch_Vertical_H20mm
- removed U1, U10, U11, U12, U13, U14, U15, U16, U18, U2, U3, U5, U6, U7, U8, U9: CherryMX_LTST-A683CEGBW, CherryMX_PCB_KailhSocket_LTST-A683CEGBW-Rotated-HS:CherryMX_1.00u_PCB_KailhSocket_LTST-A683CEGBW-Rotated-HS
- removed U101: RP2040, MCU_RaspberryPi_and_Boards:RP2040-QFN-56
- removed U102: W25Q128JVS, Package_SO:SOIC-8_5.23x5.23mm_P1.27mm
- removed U103: AMS1117-3.3, Package_TO_SOT_SMD:SOT-223-3_TabPin2
- removed U17: CherryMX_LTST-A683CEGBW, CherryMX_PCB_KailhSocket_StabWireBottom_LTST-A683CEGBW-Rotated-HS:CherryMX_2.00u_PCB_KailhSocket_StabWireBottom_LTST-A6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
- removed Y1: 12MHz, Crystal:Crystal_SMD_3225-4Pin_3.2x2.5mm
Routing:
- net +3V3: track 633.2 -> 0.00 mm, vias 26 -> 0
- net ROW4: track 173.8 -> 0.00 mm, vias 6 -> 0
- net ROW3: track 163.9 -> 0.00 mm, vias 7 -> 0
- net ROW5: track 150.2 -> 0.00 mm, vias 2 -> 0
- net COL1: track 131.7 -> 0.00 mm, vias 2 -> 0
- net COL4: track 129.6 -> 0.00 mm, vias 2 -> 0
- net ROW2: track 128.9 -> 0.00 mm, vias 5 -> 0
- net ROW1: track 104.0 -> 0.00 mm, vias 4 -> 0
- net COL3: track 101.9 -> 0.00 mm, vias 2 -> 0
- net GND: track 94.9 -> 0.00 mm, vias 55 -> 0
- net RGBData4: track 93.4 -> 0.00 mm, vias 2 -> 0
- net COL2: track 91.0 -> 0.00 mm, vias 2 -> 0
- net RGBData2: track 84.8 -> 0.00 mm, vias 2 -> 0
- net RGBData3: track 79.7 -> 0.00 mm, vias 2 -> 0
- net RGBData5: track 70.6 -> 0.00 mm, vias 2 -> 0
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- added copper zone on B.Cu, net (none)
- added copper zone on F.Cu, net (none)
- removed copper zone on B.Cu, net GND
- removed copper zone on F.Cu, net GND
Other:
- outline, holes or cut-outs redrawn
- board text added: "JLCJLCJLCJLC"
- board text removed: "BOOT RUN"
- board text removed: "CERN-OHL-W (CERN OHL v2) 2021-11-21 Pierre Constantineau"
- board text removed: "PyKey18 Numpad RP2040 Runs Python"
- board text removed: "RESET"
- board text removed: "SWD GND CLK"
- board text removed: "https://github.com/jpconstantineau/PyKey60"
