File: pykey18/switch-plate/PyKey18/PyKey18.sch (KiCad schematic (older format))
At the start: 47 parts, among them SW4 Rotary_Encoder_Switch, U1 CherryMX_LTST-A683CEGBW, U10 CherryMX_LTST-A683CEGBW, U11 CherryMX_LTST-A683CEGBW, U12 CherryMX_LTST-A683CEGBW, U13 CherryMX_LTST-A683CEGBW, U14 CherryMX_LTST-A683CEGBW, U15 CherryMX_LTST-A683CEGBW, U16 CherryMX_LTST-A683CEGBW, U17 CherryMX_LTST-A683CEGBW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

Commit message: updates to pykey87
Parts:
- removed D1, D10, D11, D12, D13, D14, D15, D16, D17, D18, D2, D3, D4, D5, D6, D7, D8, D9: D, Diode_SMD:D_SOD-123, symbol Device:D
- removed H1, H2, H3, H4: MountingHole, MountingHole:MountingHole_2.2mm_M2_DIN965, symbol Mechanical:MountingHole
- removed H10, H11: PCBA, JLCPCBA:PCBA Hole, symbol Mechanical:MountingHole
- removed H5, H6: MountingHole-feet, MountingHole:MountingHole_4.3mm_M4, symbol Mechanical:MountingHole
- removed H7: Logo, lib:KB_BlueMicro, symbol Mechanical:MountingHole
- removed H8, H9: Stabs, CherryMX_StabWireBottom:CherryMX_2.00u_StabWireBottom-nokey, symbol Mechanical:MountingHole
- U1, U10, U11, U13, U14, U15, U18, U2, U3, U5, U6, U7, U8, U9: footprint CherryMX_PCB_KailhSocket_LTST-A683CEGBW-Rotated-HS:CherryMX_1.00u_PCB_KailhSocket_LTST-A683CEGBW-Rotated-HS -> lib:Hybrid_Plate_100H
- U12, U16: footprint CherryMX_PCB_KailhSocket_LTST-A683CEGBW-Rotated-HS:CherryMX_1.00u_PCB_KailhSocket_LTST-A683CEGBW-Rotated-HS -> lib:Hybrid_Plate_200V
- U17: footprint CherryMX_PCB_KailhSocket_StabWireBottom_LTST-A683CEGBW-Rotated-HS:CherryMX_2.00u_PCB_KailhSocket_StabWireBottom_LTST-A6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 -> lib:Hybrid_Plate_200H
