File: pykey87/Bottom-plate/PyKey87-bottom.kicad_pcb (KiCad board)
At the start: 2 copper layers, 353 x 120 mm, 12 parts

Commit message: Moving things around
Prep for merging. Also did some clean up and added 8th standoff.
Parts:
- removed REF**: LED_0603_1608Metric, LED_SMD:LED_0603_1608Metric
- removed REF**: SW_Push_SPST_NO_Alps_SKRK, Button_Switch_SMD:SW_Push_SPST_NO_Alps_SKRK
- removed REF**: SW_SPDT_PCM12, Button_Switch_SMD:SW_SPDT_PCM12
- added H8: MountingHole_Pad, MountingHole:MountingHole_2.2mm_M2_Pad, F.Cu at (190.4, 110.0)
- renumbered H9 to H10, H8 to H9

Commit message: Update PyKey87-bottom.kicad_pcb
Other:
- outline, holes or cut-outs redrawn
- board text added: "Boot Run"
- board text removed: "Run Boot"
Changed lines of the file:
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@@
   (general
     (thickness 1.6)
-    (drawings 14)
+    (drawings 10)
     (tracks 0)
     (zones 0)
@@
       (net 9 "Net-(H9-Pad1)"))
   )
-  (gr_text Reset (at 91.44 119.57) (layer B.Cu)
+  (gr_text Reset (at 124.46 43.18) (layer B.Cu)
     (effects (font (size 1 1) (thickness 0.15)) (justify mirror))
   )
-  (gr_text "Run    Boot" (at 91.44 103.64) (layer B.Cu)
+  (gr_text "Boot    Run" (at 101.6 43.18) (layer B.Cu)
     (effects (font (size 1 1) (thickness 0.15)) (justify mirror))
   )
-  (gr_line (start 87.47 104.7) (end 87.47 118.7) (layer Edge.Cuts) (width 0.12))
-  (gr_line (start 95.47 104.7) (end 87.47 104.7) (layer Edge.Cuts) (width 0.12))
-  (gr_line (start 95.47 118.7) (end 95.47 104.7) (layer Edge.Cuts) (width 0.12))
-  (gr_line (start 87.47 118.7) (end 95.47 118.7) (layer Edge.Cuts) (width 0.12))
   (gr_arc (start 61 158) (end 61 160) (angle 90) (layer Edge.Cuts) (width 0.09906))
   (gr_arc (start 60.96 42) (end 58.96 42) (angle 90) (layer Edge.Cuts) (width 0.09906))

Commit message: Add logo and copper plane
Connections:
- H1 pad : Net-(H1-Pad1) -> (no net)
- H10 pad : Net-(H10-Pad1) -> (no net)
- H2 pad : Net-(H2-Pad1) -> (no net)
- H3 pad : Net-(H3-Pad1) -> (no net)
- H4 pad : Net-(H4-Pad1) -> (no net)
- H5 pad : Net-(H5-Pad1) -> (no net)
- H6 pad : Net-(H6-Pad1) -> (no net)
- H7 pad : Net-(H7-Pad1) -> (no net)
- H8 pad : Net-(H8-Pad1) -> (no net)
- H9 pad : Net-(H9-Pad1) -> (no net)
Routing:
- added copper zone on F.Cu, net (none)
